Commit message: [refac] simplify urdf joint/link names

File: urdf/mimic/pipette_macro.xacro (robot description, xacro)
@@ -3,5 +3,5 @@
   <xacro:macro name="mimic_pipette" params="prefix">
     <!-- TODO measure or calculate -->
-    <link name="${prefix}mounting_plate">
+    <link name="${prefix}base">
       <inertial>
         <origin xyz="0 0 0" rpy="0 0 0" />
@@ -32,7 +32,7 @@
     </link>
     <link name="${prefix}tcp" />
-    <joint name="${prefix}mounting_plate_joint" type="fixed">
+    <joint name="${prefix}tcp_joint" type="fixed">
       <origin xyz="0.25344 0 0" rpy="0 0 0" />
-      <parent link="${prefix}mounting_plate" />
+      <parent link="${prefix}base" />
       <child link="${prefix}tcp" />
     </joint>

File: urdf/mimic/ur3_mounting_plate_macro.xacro (robot description, xacro)
@@ -2,5 +2,5 @@
 <robot name="mimic_ur3_mounting_plate" xmlns:xacro="http://www.ros.org/wiki/xacro">
   <xacro:macro name="mimic_ur3_mounting_plate" params="prefix">
-    <link name="${prefix}plate_base">
+    <link name="${prefix}base">
       <inertial>
         <origin xyz="0 0 0" rpy="0 0 0" />
@@ -31,10 +31,10 @@
       </collision>
     </link>
-    <link name="${prefix}plate" />
+    <link name="${prefix}robotside" />
     <!-- Mean of multiple points of the surface -->
-    <joint name="${prefix}plate_joint" type="fixed">
+    <joint name="${prefix}robotside_joint" type="fixed">
       <origin xyz="0 0 0.01309" rpy="0 0 0" />
-      <parent link="${prefix}plate_base" />
-      <child link="${prefix}plate" />
+      <parent link="${prefix}base" />
+      <child link="${prefix}robotside" />
     </joint>
   </xacro:macro>

File: urdf/ur3_dual_eef_wc_mobile.xacro (robot description, xacro)
@@ -4,4 +4,5 @@
   <xacro:include filename="$(find mimic_description)/urdf/mimic/ur3_mounting_plate_macro.xacro"/>
   <xacro:include filename="$(find ur_description)/urdf/inc/ur3_macro.xacro"/>
+  <xacro:include filename="$(find robotiq_description)/urdf/robotiq_fts_300_cpl_062/robotiq_fts_300_cpl_062_macro.xacro"/>
   <xacro:include filename="$(find robotiq_description)/urdf/robotiq_ft_300/robotiq_ft_300_macro.xacro"/>
   <xacro:include filename="$(find robotiq_description)/urdf/robotiq_agc_apl_159_002/robotiq_agc_apl_159_002_macro.xacro"/>
@@ -48,23 +49,27 @@
     prefix="newport_"/>
   <xacro:mimic_ur3_mounting_plate
-    prefix="ur3_mounting_"/>
+    prefix="ur3_mounting_plate_"/>
   <!-- UR3 with S/N: 2017333047 -->
   <xacro:ur3_robot
     prefix="ur3_"
     kinematics_parameters_file="$(find mimic_ur_launch)/etc/ur3-2017333047-calibration.yaml"
-    visual_parameters_file="$(find ur_description)/config/ur3/visual_parameters_bbox.yaml"/>
+    visual_parameters_file="$(find ur_description)/config/ur3/visual_parameters.yaml"/>
+  <!-- FT300 ur coupling + sensor -->
+  <xacro:robotiq_fts_300_cpl_062
+    prefix="robotiq_ft300_coupling_"
+    visual_parameters_file="$(find robotiq_description)/config/robotiq_fts_300_cpl_062/visual_parameters.yaml"/>
   <xacro:robotiq_ft_300
     prefix="robotiq_ft300_"
-    visual_parameters_file="$(find robotiq_description)/config/robotiq_ft_300/visual_parameters_bbox.yaml"/>
-  Dual gripper mounting plate
+    visual_parameters_file="$(find robotiq_description)/config/robotiq_ft_300/visual_parameters.yaml"/>
+  <!-- Dual gripper mounting plate -->
   <xacro:robotiq_agc_apl_159_002
-    prefix="dual_gripper_"
-    visual_parameters_file="$(find robotiq_description)/config/robotiq_agc_apl_159_002/visual_parameters_bbox.yaml"/>
+    prefix="dual_gripper_coupling_"
+    visual_parameters_file="$(find robotiq_description)/config/robotiq_agc_apl_159_002/visual_parameters.yaml"/>
   <xacro:robotiq_2f_140
     prefix="robotiq_2f140_"
-    visual_parameters_file="$(find robotiq_description)/config/robotiq_2f_140/visual_parameters_bbox.yaml"/>
+    visual_parameters_file="$(find robotiq_description)/config/robotiq_2f_140/visual_parameters.yaml"/>
   <xacro:mimic_pipette
     prefix="pipette_"/>
-  <joint name="tabletop_newport_tabletop_joint" type="fixed">
+  <joint name="newport_base_joint" type="fixed">
     <parent link= "tabletop" />
     <child link = "newport_base" />
@@ -72,39 +77,44 @@
     <origin xyz="0 0 ${1.5 * 0.0254 + 0.0254/2}" rpy="0.0 0.0 0.0" />
   </joint>
-  <joint name="tabletop_wall_joint" type="fixed">
+  <joint name="wall_joint" type="fixed">
     <parent link= "tabletop" />
     <child link = "wall" />
     <origin xyz="0 ${-(22 * 0.0254 - 0.0254/2)} ${44*0.0254/2}" rpy="0.0 0.0 0.0" />
   </joint>
-  <joint name="newport_tabletop_ur3_mounting_plate_coupling" type="fixed">
+  <joint name="ur3_mounting_plate_base_joint" type="fixed">
     <parent link= "newport_tabletop" />
     <child link = "ur3_mounting_plate_base" />
-    <!-- Tabletop has matrix of 1" hole gap-->
-    <origin xyz="${-10*0.0254} ${-12*0.0254} 0.0" rpy="0.0 0.0 0.0" />
+    <!-- Newport tabletop has matrix of 1 inch hole gap-->
+    <origin xyz="${-10 * 0.0254} ${-12 * 0.0254} 0.0" rpy="0.0 0.0 0.0" />
   </joint>
-  <joint name="ur3_mounting_plate_ur3_coupling" type="fixed">
-    <parent link= "ur3_mounting_plate" />
+  <joint name="ur3_base_joint" type="fixed">
+    <parent link= "ur3_mounting_plate_robotside" />
     <child link = "ur3_base_link" />
     <origin xyz="0.0 0.0 0.0" rpy="0.0 0.0 0.0" />
   </joint>
-  <joint name="ur3_robotiqft300_coupling" type="fixed">
+  <joint name="robotiq_fts300_coupling_joint" type="fixed">
     <parent link= "ur3_flange" />
-    <child link = "robotiq_ft300_mounting_plate" />
+    <child link = "robotiq_ft300_coupling_robotside" />
     <!-- Align mounting plate to flange -->
     <origin xyz="0.0 0.0 0.0" rpy="${pi} 0.0 0.0" />
   </joint>
-  <joint name="robotiqft300_dual_gripper_coupling" type="fixed">
-    <parent link= "robotiq_ft300_sensor" />
-    <child link = "dual_gripper_mounting_plate" />
+  <joint name="robotiq_ft300_joint" type="fixed">
+    <parent link= "robotiq_ft300_coupling_toolside" />
+    <child link = "robotiq_ft300_robotside" />
+    <origin xyz="0.0 0.0 0.0" rpy="0 0.0 0.0" />
+  </joint>
+  <joint name="dual_gripper_coupling_robotside_joint" type="fixed">
+    <parent link= "robotiq_ft300_toolside" />
+    <child link = "dual_gripper_coupling_robotside" />
     <origin xyz="0.0 0.0 0.0" rpy="0.0 0.0 0.0" />
   </joint>
-  <joint name="dual_gripper_left_flange_robotiq140_coupling" type="fixed">
-    <parent link= "dual_gripper_left_flange" />
+  <joint name="robotiq_2f140_base_joint" type="fixed">
+    <parent link= "dual_gripper_coupling_toolside_left" />
     <child link = "robotiq_2f140_base_link" />
     <origin xyz="0.0 0.0 0.0" rpy="0.0 0.0 0.0" />
   </joint>
-  <joint name="dual_gripper_right_flange_pipette_coupling" type="fixed">
-    <parent link= "dual_gripper_right_flange" />
-    <child link = "pipette_mounting_plate" />
+  <joint name="pipette_base_joint" type="fixed">
+    <parent link= "dual_gripper_coupling_toolside_right" />
+    <child link = "pipette_base" />
     <origin xyz="0.0 0.0 0.0" rpy="0.0 0.0 0.0" />
   </joint>
