Commit message: [refac] update filenames to new convention

File: urdf/biorad/thermal_cycler_t100_open_macro.xacro (robot description, xacro)
@@ -1,10 +1,9 @@
 <?xml version="1.0"?>
-<robot name="calibration_adapter_robotiq2f140" xmlns:xacro="http://www.ros.org/wiki/xacro">
-  <xacro:macro name="calibration_adapter_robotiq2f140" params="prefix">
+<robot name="thermal_cycler_t100_open" xmlns:xacro="http://www.ros.org/wiki/xacro">
+  <xacro:macro name="thermal_cycler_t100_open" params="prefix">
     <link name="${prefix}base">
       <inertial>
         <origin xyz="0 0 0" rpy="0 0 0" />
-        <!-- Not measured -->
-        <mass value="0.5" />
+        <mass value="19.86735" />
         <inertia
           ixx="0"
@@ -18,5 +17,5 @@
         <origin xyz="0 0 0" rpy="0 0 0" />
         <geometry>
-          <mesh filename="package://mimic_description/meshes/mimic/visual/calibration_adapter_robotiq2f140.dae"/>
+          <mesh filename="package://mimic_description/meshes/biorad/thermal_cycler_t100/visual/full_open_226k.dae"/>
         </geometry>
         <material name="">
@@ -27,5 +26,5 @@
         <origin xyz="0 0 0" rpy="0 0 0" />
         <geometry>
-          <mesh filename="package://mimic_description/meshes/mimic/collision/calibration_adapter_robotiq2f140.stl"/>
+          <mesh filename="package://mimic_description/meshes/biorad/thermal_cycler_t100/collision/full_open_226k.stl"/>
         </geometry>
       </collision>

File: urdf/mimic/biorad_t100_adapter_macro.xacro (robot description, xacro)
@@ -1,9 +1,10 @@
 <?xml version="1.0"?>
-<robot name="newport_sa2_30x30" xmlns:xacro="http://www.ros.org/wiki/xacro">
-  <xacro:macro name="newport_sa2_30x30" params="prefix">
+<robot name="mimic_biorad_t100_adapter" xmlns:xacro="http://www.ros.org/wiki/xacro">
+  <xacro:macro name="mimic_biorad_t100_adapter" params="prefix">
+    <!-- TODO measure or calculate -->
     <link name="${prefix}base">
       <inertial>
         <origin xyz="0 0 0" rpy="0 0 0" />
-        <mass value="19.86735" />
+        <mass value="0.5" />
         <inertia
           ixx="0"
@@ -17,5 +18,5 @@
         <origin xyz="0 0 0" rpy="0 0 0" />
         <geometry>
-		<mesh filename="package://mimic_description/meshes/newport/sa2_30x30/visual/101k.dae"/>
+          <mesh filename="package://mimic_description/meshes/mimic/biorad_t100_adapter/visual/50k.dae"/>
         </geometry>
         <material name="">
@@ -26,14 +27,8 @@
         <origin xyz="0 0 0" rpy="0 0 0" />
         <geometry>
-		<mesh filename="package://mimic_description/meshes/newport/sa2_30x30/collision/p12.stl"/>
+          <mesh filename="package://mimic_description/meshes/mimic/biorad_t100_adapter/collision/50k.stl"/>
         </geometry>
       </collision>
     </link>
-    <link name="${prefix}tabletop" />
-    <joint name="${prefix}tabletop_joint" type="fixed">
-      <origin xyz="0 0 0.0127" rpy="0 0 0" />
-      <parent link="${prefix}base" />
-      <child link="${prefix}tabletop" />
-    </joint>
   </xacro:macro>
 </robot>

File: urdf/mimic/pipette_p200_macro.xacro (robot description, xacro)
@@ -1,7 +1,7 @@
 <?xml version="1.0"?>
-<robot name="mimic_capture_tool" xmlns:xacro="http://www.ros.org/wiki/xacro">
-  <xacro:macro name="mimic_capture_tool" params="prefix">
+<robot name="mimic_pipette_p200" xmlns:xacro="http://www.ros.org/wiki/xacro">
+  <xacro:macro name="mimic_pipette_p200" params="prefix">
     <!-- TODO measure or calculate -->
-    <link name="${prefix}robotside">
+    <link name="${prefix}base">
       <inertial>
         <origin xyz="0 0 0" rpy="0 0 0" />
@@ -18,5 +18,5 @@
         <origin xyz="0 0 0" rpy="0 0 0" />
         <geometry>
-          <mesh filename="package://mimic_description/meshes/mimic/visual/capture_tool.dae"/>
+          <mesh filename="package://mimic_description/meshes/mimic/pipette_p200/visual/9k.dae"/>
         </geometry>
         <material name="">
@@ -27,5 +27,5 @@
         <origin xyz="0 0 0" rpy="0 0 0" />
         <geometry>
-          <mesh filename="package://mimic_description/meshes/mimic/collision/capture_tool.stl"/>
+          <mesh filename="package://mimic_description/meshes/mimic/pipette_p200/collision/p36.stl"/>
         </geometry>
       </collision>
@@ -33,6 +33,6 @@
     <link name="${prefix}tcp" />
     <joint name="${prefix}tcp_joint" type="fixed">
-      <origin xyz="0.0745 0 0" rpy="0 0 0" />
-      <parent link="${prefix}robotside" />
+      <origin xyz="0.25344 0 0" rpy="0 0 0" />
+      <parent link="${prefix}base" />
       <child link="${prefix}tcp" />
     </joint>

File: urdf/mimic/robotiq_2f140_calibration_adapter_macro.xacro (robot description, xacro)
@@ -1,5 +1,5 @@
 <?xml version="1.0"?>
-<robot name="mimic_ur3_mounting_plate" xmlns:xacro="http://www.ros.org/wiki/xacro">
-  <xacro:macro name="mimic_ur3_mounting_plate" params="prefix">
+<robot name="mimic_robotiq_2f140_calibration_adapter" xmlns:xacro="http://www.ros.org/wiki/xacro">
+  <xacro:macro name="mimic_robotiq_2f140_calibration_adapter" params="prefix">
     <link name="${prefix}base">
       <inertial>
@@ -18,5 +18,5 @@
         <origin xyz="0 0 0" rpy="0 0 0" />
         <geometry>
-          <mesh filename="package://mimic_description/meshes/mimic/ur3_mounting_plate/visual/2k.dae"/>
+          <mesh filename="package://mimic_description/meshes/mimic/robotiq_2f140_calibration_adapter/visual/928.dae"/>
         </geometry>
         <material name="">
@@ -27,15 +27,8 @@
         <origin xyz="0 0 0" rpy="0 0 0" />
         <geometry>
-          <mesh filename="package://mimic_description/meshes/mimic/ur3_mounting_plate/collision/cv12.stl"/>
+          <mesh filename="package://mimic_description/meshes/mimic/robotiq_2f140_calibration_adapter/collision/928.stl"/>
         </geometry>
       </collision>
     </link>
-    <link name="${prefix}robotside" />
-    <!-- Mean of multiple points of the surface -->
-    <joint name="${prefix}robotside_joint" type="fixed">
-      <origin xyz="0 0 0.01309" rpy="0 0 0" />
-      <parent link="${prefix}base" />
-      <child link="${prefix}robotside" />
-    </joint>
   </xacro:macro>
 </robot>

File: urdf/mimic/ur3_capture_tool_macro.xacro (robot description, xacro)
@@ -1,7 +1,7 @@
 <?xml version="1.0"?>
-<robot name="mimic_pipette" xmlns:xacro="http://www.ros.org/wiki/xacro">
-  <xacro:macro name="mimic_pipette" params="prefix">
+<robot name="mimic_ur3_capture_tool" xmlns:xacro="http://www.ros.org/wiki/xacro">
+  <xacro:macro name="mimic_ur3_capture_tool" params="prefix">
     <!-- TODO measure or calculate -->
-    <link name="${prefix}base">
+    <link name="${prefix}robotside">
       <inertial>
         <origin xyz="0 0 0" rpy="0 0 0" />
@@ -18,5 +18,5 @@
         <origin xyz="0 0 0" rpy="0 0 0" />
         <geometry>
-          <mesh filename="package://mimic_description/meshes/mimic/visual/pipette_simple.dae"/>
+          <mesh filename="package://mimic_description/meshes/mimic/ur3_capture_tool/visual/1k.dae"/>
         </geometry>
         <material name="">
@@ -27,5 +27,5 @@
         <origin xyz="0 0 0" rpy="0 0 0" />
         <geometry>
-          <mesh filename="package://mimic_description/meshes/mimic/collision/pipette.stl"/>
+          <mesh filename="package://mimic_description/meshes/mimic/ur3_capture_tool/collision/1k.stl"/>
         </geometry>
       </collision>
@@ -33,6 +33,6 @@
     <link name="${prefix}tcp" />
     <joint name="${prefix}tcp_joint" type="fixed">
-      <origin xyz="0.25344 0 0" rpy="0 0 0" />
-      <parent link="${prefix}base" />
+      <origin xyz="0.0745 0 0" rpy="0 0 0" />
+      <parent link="${prefix}robotside" />
       <child link="${prefix}tcp" />
     </joint>

Commit message: [impl] add biorad thermal cycler t100

File: urdf/biorad/thermal_cycler_t100_open_macro.xacro (robot description, xacro)
@@ -1,5 +1,5 @@
 <?xml version="1.0"?>
-<robot name="thermal_cycler_t100_open" xmlns:xacro="http://www.ros.org/wiki/xacro">
-  <xacro:macro name="thermal_cycler_t100_open" params="prefix">
+<robot name="biorad_thermal_cycler_t100_open" xmlns:xacro="http://www.ros.org/wiki/xacro">
+  <xacro:macro name="biorad_thermal_cycler_t100_open" params="prefix">
     <link name="${prefix}base">
       <inertial>

Commit message: [refac] rename mimic to mimik

File: urdf/biorad/thermal_cycler_t100_open_macro.xacro (robot description, xacro)
@@ -17,5 +17,5 @@
         <origin xyz="0 0 0" rpy="0 0 0" />
         <geometry>
-          <mesh filename="package://mimic_description/meshes/biorad/thermal_cycler_t100/visual/full_open_226k.dae"/>
+          <mesh filename="package://mimik_description/meshes/biorad/thermal_cycler_t100/visual/full_open_226k.dae"/>
         </geometry>
         <material name="">
@@ -26,5 +26,5 @@
         <origin xyz="0 0 0" rpy="0 0 0" />
         <geometry>
-          <mesh filename="package://mimic_description/meshes/biorad/thermal_cycler_t100/collision/full_open_226k.stl"/>
+          <mesh filename="package://mimik_description/meshes/biorad/thermal_cycler_t100/collision/full_open_226k.stl"/>
         </geometry>
       </collision>

File: urdf/mimik/biorad_t100_adapter_macro.xacro (robot description, xacro)
@@ -1,5 +1,5 @@
 <?xml version="1.0"?>
-<robot name="mimic_biorad_t100_adapter" xmlns:xacro="http://www.ros.org/wiki/xacro">
-  <xacro:macro name="mimic_biorad_t100_adapter" params="prefix">
+<robot name="mimik_biorad_t100_adapter" xmlns:xacro="http://www.ros.org/wiki/xacro">
+  <xacro:macro name="mimik_biorad_t100_adapter" params="prefix">
     <!-- TODO measure or calculate -->
     <link name="${prefix}base">
@@ -18,5 +18,5 @@
         <origin xyz="0 0 0" rpy="0 0 0" />
         <geometry>
-          <mesh filename="package://mimic_description/meshes/mimic/biorad_t100_adapter/visual/50k.dae"/>
+          <mesh filename="package://mimik_description/meshes/mimik/biorad_t100_adapter/visual/50k.dae"/>
         </geometry>
         <material name="">
@@ -27,5 +27,5 @@
         <origin xyz="0 0 0" rpy="0 0 0" />
         <geometry>
-          <mesh filename="package://mimic_description/meshes/mimic/biorad_t100_adapter/collision/50k.stl"/>
+          <mesh filename="package://mimik_description/meshes/mimik/biorad_t100_adapter/collision/50k.stl"/>
         </geometry>
       </collision>

File: urdf/mimik/pipette_p200_macro.xacro (robot description, xacro)
@@ -1,9 +1,9 @@
 <?xml version="1.0"?>
-<robot name="mimic_robotiq_2f140_calibration_adapter" xmlns:xacro="http://www.ros.org/wiki/xacro">
-  <xacro:macro name="mimic_robotiq_2f140_calibration_adapter" params="prefix">
+<robot name="mimik_pipette_p200" xmlns:xacro="http://www.ros.org/wiki/xacro">
+  <xacro:macro name="mimik_pipette_p200" params="prefix">
+    <!-- TODO measure or calculate -->
     <link name="${prefix}base">
       <inertial>
         <origin xyz="0 0 0" rpy="0 0 0" />
-        <!-- Not measured -->
         <mass value="0.5" />
         <inertia
@@ -18,5 +18,5 @@
         <origin xyz="0 0 0" rpy="0 0 0" />
         <geometry>
-          <mesh filename="package://mimic_description/meshes/mimic/robotiq_2f140_calibration_adapter/visual/928.dae"/>
+          <mesh filename="package://mimik_description/meshes/mimik/pipette_p200/visual/9k.dae"/>
         </geometry>
         <material name="">
@@ -27,8 +27,14 @@
         <origin xyz="0 0 0" rpy="0 0 0" />
         <geometry>
-          <mesh filename="package://mimic_description/meshes/mimic/robotiq_2f140_calibration_adapter/collision/928.stl"/>
+          <mesh filename="package://mimik_description/meshes/mimik/pipette_p200/collision/p36.stl"/>
         </geometry>
       </collision>
     </link>
+    <link name="${prefix}tcp" />
+    <joint name="${prefix}tcp_joint" type="fixed">
+      <origin xyz="0.25344 0 0" rpy="0 0 0" />
+      <parent link="${prefix}base" />
+      <child link="${prefix}tcp" />
+    </joint>
   </xacro:macro>
 </robot>

File: urdf/mimik/robotiq_2f140_calibration_adapter_macro.xacro (robot description, xacro)
@@ -1,9 +1,9 @@
 <?xml version="1.0"?>
-<robot name="mimic_pipette_p200" xmlns:xacro="http://www.ros.org/wiki/xacro">
-  <xacro:macro name="mimic_pipette_p200" params="prefix">
-    <!-- TODO measure or calculate -->
+<robot name="mimik_robotiq_2f140_calibration_adapter" xmlns:xacro="http://www.ros.org/wiki/xacro">
+  <xacro:macro name="mimik_robotiq_2f140_calibration_adapter" params="prefix">
     <link name="${prefix}base">
       <inertial>
         <origin xyz="0 0 0" rpy="0 0 0" />
+        <!-- Not measured -->
         <mass value="0.5" />
         <inertia
@@ -18,5 +18,5 @@
         <origin xyz="0 0 0" rpy="0 0 0" />
         <geometry>
-          <mesh filename="package://mimic_description/meshes/mimic/pipette_p200/visual/9k.dae"/>
+          <mesh filename="package://mimik_description/meshes/mimik/robotiq_2f140_calibration_adapter/visual/928.dae"/>
         </geometry>
         <material name="">
@@ -27,14 +27,8 @@
         <origin xyz="0 0 0" rpy="0 0 0" />
         <geometry>
-          <mesh filename="package://mimic_description/meshes/mimic/pipette_p200/collision/p36.stl"/>
+          <mesh filename="package://mimik_description/meshes/mimik/robotiq_2f140_calibration_adapter/collision/928.stl"/>
         </geometry>
       </collision>
     </link>
-    <link name="${prefix}tcp" />
-    <joint name="${prefix}tcp_joint" type="fixed">
-      <origin xyz="0.25344 0 0" rpy="0 0 0" />
-      <parent link="${prefix}base" />
-      <child link="${prefix}tcp" />
-    </joint>
   </xacro:macro>
 </robot>

File: urdf/mimik/ur3_capture_tool_macro.xacro (robot description, xacro)
@@ -1,5 +1,5 @@
 <?xml version="1.0"?>
-<robot name="mimic_ur3_capture_tool" xmlns:xacro="http://www.ros.org/wiki/xacro">
-  <xacro:macro name="mimic_ur3_capture_tool" params="prefix">
+<robot name="mimik_ur3_capture_tool" xmlns:xacro="http://www.ros.org/wiki/xacro">
+  <xacro:macro name="mimik_ur3_capture_tool" params="prefix">
     <!-- TODO measure or calculate -->
     <link name="${prefix}robotside">
@@ -18,5 +18,5 @@
         <origin xyz="0 0 0" rpy="0 0 0" />
         <geometry>
-          <mesh filename="package://mimic_description/meshes/mimic/ur3_capture_tool/visual/1k.dae"/>
+          <mesh filename="package://mimik_description/meshes/mimik/ur3_capture_tool/visual/1k.dae"/>
         </geometry>
         <material name="">
@@ -27,5 +27,5 @@
         <origin xyz="0 0 0" rpy="0 0 0" />
         <geometry>
-          <mesh filename="package://mimic_description/meshes/mimic/ur3_capture_tool/collision/1k.stl"/>
+          <mesh filename="package://mimik_description/meshes/mimik/ur3_capture_tool/collision/1k.stl"/>
         </geometry>
       </collision>

File: urdf/mimik/ur3_mounting_plate_macro.xacro (robot description, xacro)
@@ -1,5 +1,5 @@
 <?xml version="1.0"?>
-<robot name="mimic_ur3_mounting_plate" xmlns:xacro="http://www.ros.org/wiki/xacro">
-  <xacro:macro name="mimic_ur3_mounting_plate" params="prefix">
+<robot name="mimik_ur3_mounting_plate" xmlns:xacro="http://www.ros.org/wiki/xacro">
+  <xacro:macro name="mimik_ur3_mounting_plate" params="prefix">
     <link name="${prefix}base">
       <inertial>
@@ -18,5 +18,5 @@
         <origin xyz="0 0 0" rpy="0 0 0" />
         <geometry>
-          <mesh filename="package://mimic_description/meshes/mimic/ur3_mounting_plate/visual/2k.dae"/>
+          <mesh filename="package://mimik_description/meshes/mimik/ur3_mounting_plate/visual/2k.dae"/>
         </geometry>
         <material name="">
@@ -27,5 +27,5 @@
         <origin xyz="0 0 0" rpy="0 0 0" />
         <geometry>
-          <mesh filename="package://mimic_description/meshes/mimic/ur3_mounting_plate/collision/cv12.stl"/>
+          <mesh filename="package://mimik_description/meshes/mimik/ur3_mounting_plate/collision/cv12.stl"/>
         </geometry>
       </collision>

File: urdf/newport/sa2_30x30_macro.xacro (robot description, xacro)
@@ -17,5 +17,5 @@
         <origin xyz="0 0 0" rpy="0 0 0" />
         <geometry>
-		<mesh filename="package://mimic_description/meshes/newport/sa2_30x30/visual/101k.dae"/>
+		<mesh filename="package://mimik_description/meshes/newport/sa2_30x30/visual/101k.dae"/>
         </geometry>
         <material name="">
@@ -26,5 +26,5 @@
         <origin xyz="0 0 0" rpy="0 0 0" />
         <geometry>
-		<mesh filename="package://mimic_description/meshes/newport/sa2_30x30/collision/p12.stl"/>
+		<mesh filename="package://mimik_description/meshes/newport/sa2_30x30/collision/p12.stl"/>
         </geometry>
       </collision>
