Commit message: [refac] renamed to thermocycler

File: urdf/biorad/thermocycler_t100_open_macro.xacro (robot description, xacro)
@@ -1,5 +1,5 @@
 <?xml version="1.0"?>
-<robot name="biorad_thermal_cycler_t100_open" xmlns:xacro="http://www.ros.org/wiki/xacro">
-  <xacro:macro name="biorad_thermal_cycler_t100_open" params="prefix">
+<robot name="biorad_thermocycler_t100_open" xmlns:xacro="http://www.ros.org/wiki/xacro">
+  <xacro:macro name="biorad_thermocycler_t100_open" params="prefix">
     <link name="${prefix}base">
       <inertial>
@@ -17,5 +17,5 @@
         <origin xyz="0 0 0" rpy="0 0 0" />
         <geometry>
-          <mesh filename="package://mimik_description/meshes/biorad/thermal_cycler_t100/visual/full_open_226k.dae"/>
+          <mesh filename="package://mimik_description/meshes/biorad/thermocycler_t100/visual/full_open_226k.dae"/>
         </geometry>
         <material name="">
@@ -26,5 +26,5 @@
         <origin xyz="0 0 0" rpy="0 0 0" />
         <geometry>
-          <mesh filename="package://mimik_description/meshes/biorad/thermal_cycler_t100/collision/full_open_226k.stl"/>
+          <mesh filename="package://mimik_description/meshes/biorad/thermocycler_t100/collision/full_open_226k.stl"/>
         </geometry>
       </collision>

Commit message: [refac] renamed package

File: urdf/biorad/thermocycler_t100_open_macro.xacro (robot description, xacro)
@@ -17,5 +17,5 @@
         <origin xyz="0 0 0" rpy="0 0 0" />
         <geometry>
-          <mesh filename="package://mimik_description/meshes/biorad/thermocycler_t100/visual/full_open_226k.dae"/>
+          <mesh filename="package://oscar_description/meshes/biorad/thermocycler_t100/visual/full_open_226k.dae"/>
         </geometry>
         <material name="">
@@ -26,5 +26,5 @@
         <origin xyz="0 0 0" rpy="0 0 0" />
         <geometry>
-          <mesh filename="package://mimik_description/meshes/biorad/thermocycler_t100/collision/full_open_226k.stl"/>
+          <mesh filename="package://oscar_description/meshes/biorad/thermocycler_t100/collision/full_open_226k.stl"/>
         </geometry>
       </collision>

File: urdf/intel/realsense_d415_macro.xacro (robot description, xacro)
@@ -18,5 +18,5 @@
         <origin xyz="0 0 0" rpy="0 0 0" />
         <geometry>
-          <mesh filename="package://mimik_description/meshes/intel/realsense_d415/visual/23k.dae"/>
+          <mesh filename="package://oscar_description/meshes/intel/realsense_d415/visual/23k.dae"/>
         </geometry>
         <material name="">
@@ -27,5 +27,5 @@
         <origin xyz="0 0 0" rpy="0 0 0" />
         <geometry>
-          <mesh filename="package://mimik_description/meshes/intel/realsense_d415/collision/p12.stl"/>
+          <mesh filename="package://oscar_description/meshes/intel/realsense_d415/collision/p12.stl"/>
         </geometry>
       </collision>

File: urdf/newport/sa2_30x30_macro.xacro (robot description, xacro)
@@ -17,5 +17,5 @@
         <origin xyz="0 0 0" rpy="0 0 0" />
         <geometry>
-		<mesh filename="package://mimik_description/meshes/newport/sa2_30x30/visual/101k.dae"/>
+		<mesh filename="package://oscar_description/meshes/newport/sa2_30x30/visual/101k.dae"/>
         </geometry>
         <material name="">
@@ -26,5 +26,5 @@
         <origin xyz="0 0 0" rpy="0 0 0" />
         <geometry>
-		<mesh filename="package://mimik_description/meshes/newport/sa2_30x30/collision/p12.stl"/>
+		<mesh filename="package://oscar_description/meshes/newport/sa2_30x30/collision/p12.stl"/>
         </geometry>
       </collision>

File: urdf/picknik/ur5_realsense_camera_adapter_macro.xacro (robot description, xacro)
@@ -17,5 +17,5 @@
         <origin xyz="0 0 0" rpy="0 0 0" />
         <geometry>
-          <mesh filename="package://mimik_description/meshes/picknik/ur5_realsense_camera_adapter/visual/28k.dae"/>
+          <mesh filename="package://oscar_description/meshes/picknik/ur5_realsense_camera_adapter/visual/28k.dae"/>
         </geometry>
         <material name="">
@@ -26,5 +26,5 @@
         <origin xyz="0 0 0" rpy="0 0 0" />
         <geometry>
-          <mesh filename="package://mimik_description/meshes/picknik/ur5_realsense_camera_adapter/collision/p12.stl"/>
+          <mesh filename="package://oscar_description/meshes/picknik/ur5_realsense_camera_adapter/collision/p12.stl"/>
         </geometry>
       </collision>

File: urdf/udes/biorad_t100_adapter_macro.xacro (robot description, xacro)
@@ -1,5 +1,5 @@
 <?xml version="1.0"?>
-<robot name="mimik_biorad_t100_adapter" xmlns:xacro="http://www.ros.org/wiki/xacro">
-  <xacro:macro name="mimik_biorad_t100_adapter" params="prefix">
+<robot name="udes_biorad_t100_adapter" xmlns:xacro="http://www.ros.org/wiki/xacro">
+  <xacro:macro name="udes_biorad_t100_adapter" params="prefix">
     <!-- TODO measure or calculate -->
     <link name="${prefix}base">
@@ -18,5 +18,5 @@
         <origin xyz="0 0 0" rpy="0 0 0" />
         <geometry>
-          <mesh filename="package://mimik_description/meshes/mimik/biorad_t100_adapter/visual/50k.dae"/>
+          <mesh filename="package://oscar_description/meshes/udes/biorad_t100_adapter/visual/50k.dae"/>
         </geometry>
         <material name="">
@@ -27,5 +27,5 @@
         <origin xyz="0 0 0" rpy="0 0 0" />
         <geometry>
-          <mesh filename="package://mimik_description/meshes/mimik/biorad_t100_adapter/collision/50k.stl"/>
+          <mesh filename="package://oscar_description/meshes/udes/biorad_t100_adapter/collision/50k.stl"/>
         </geometry>
       </collision>

File: urdf/udes/pipette_p200_macro.xacro (robot description, xacro)
@@ -1,9 +1,9 @@
 <?xml version="1.0"?>
-<robot name="mimik_robotiq_2f140_calibration_adapter" xmlns:xacro="http://www.ros.org/wiki/xacro">
-  <xacro:macro name="mimik_robotiq_2f140_calibration_adapter" params="prefix">
+<robot name="udes_pipette_p200" xmlns:xacro="http://www.ros.org/wiki/xacro">
+  <xacro:macro name="udes_pipette_p200" params="prefix">
+    <!-- TODO measure or calculate -->
     <link name="${prefix}base">
       <inertial>
         <origin xyz="0 0 0" rpy="0 0 0" />
-        <!-- Not measured -->
         <mass value="0.5" />
         <inertia
@@ -18,5 +18,5 @@
         <origin xyz="0 0 0" rpy="0 0 0" />
         <geometry>
-          <mesh filename="package://mimik_description/meshes/mimik/robotiq_2f140_calibration_adapter/visual/928.dae"/>
+          <mesh filename="package://oscar_description/meshes/udes/pipette_p200/visual/9k.dae"/>
         </geometry>
         <material name="">
@@ -27,8 +27,15 @@
         <origin xyz="0 0 0" rpy="0 0 0" />
         <geometry>
-          <mesh filename="package://mimik_description/meshes/mimik/robotiq_2f140_calibration_adapter/collision/928.stl"/>
+          <mesh filename="package://oscar_description/meshes/udes/pipette_p200/collision/pipette_p200_coarse.stl"/>
         </geometry>
       </collision>
     </link>
+    <link name="${prefix}tip" />
+    <joint name="${prefix}tip_joint" type="fixed">
+      <!-- Original CAD -->
+      <origin xyz="0.253442 0 0" rpy="0 0 0" />
+      <parent link="${prefix}base" />
+      <child link="${prefix}tip" />
+    </joint>
   </xacro:macro>
 </robot>

File: urdf/udes/realsense_camera_adapter_macro.xacro (robot description, xacro)
@@ -1,10 +1,10 @@
 <?xml version="1.0"?>
-<robot name="mimik_ur3_capture_tool" xmlns:xacro="http://www.ros.org/wiki/xacro">
-  <xacro:macro name="mimik_ur3_capture_tool" params="prefix">
+<robot name="udes_realsense_camera_adapter" xmlns:xacro="http://www.ros.org/wiki/xacro">
+  <xacro:macro name="udes_realsense_camera_adapter" params="prefix">
     <!-- TODO measure or calculate -->
     <link name="${prefix}robotside">
       <inertial>
         <origin xyz="0 0 0" rpy="0 0 0" />
-        <mass value="0.5" />
+        <mass value="0.2" />
         <inertia
           ixx="0"
@@ -18,5 +18,5 @@
         <origin xyz="0 0 0" rpy="0 0 0" />
         <geometry>
-          <mesh filename="package://mimik_description/meshes/mimik/ur3_capture_tool/visual/1k.dae"/>
+          <mesh filename="package://oscar_description/meshes/udes/realsense_camera_adapter/visual/realsense_camera_adapter_1k.dae"/>
         </geometry>
         <material name="">
@@ -27,13 +27,14 @@
         <origin xyz="0 0 0" rpy="0 0 0" />
         <geometry>
-          <mesh filename="package://mimik_description/meshes/mimik/ur3_capture_tool/collision/1k.stl"/>
+          <mesh filename="package://oscar_description/meshes/udes/realsense_camera_adapter/collision/realsense_camera_adapter_bbox.stl"/>
         </geometry>
       </collision>
     </link>
-    <link name="${prefix}tcp" />
-    <joint name="${prefix}tcp_joint" type="fixed">
-      <origin xyz="0.0745 0 0" rpy="0 0 0" />
+    <link name="${prefix}toolside" />
+    <joint name="${prefix}toolside_joint" type="fixed">
+      <!-- Original CAD -->
+      <origin xyz="0.045 0 0.016" rpy="0 0 0" />
       <parent link="${prefix}robotside" />
-      <child link="${prefix}tcp" />
+      <child link="${prefix}toolside" />
     </joint>
   </xacro:macro>

File: urdf/udes/robotiq_2f140_calibration_adapter_macro.xacro (robot description, xacro)
@@ -1,5 +1,5 @@
 <?xml version="1.0"?>
-<robot name="mimik_ur_mounting_plate" xmlns:xacro="http://www.ros.org/wiki/xacro">
-  <xacro:macro name="mimik_ur_mounting_plate" params="prefix">
+<robot name="udes_robotiq_2f140_calibration_adapter" xmlns:xacro="http://www.ros.org/wiki/xacro">
+  <xacro:macro name="udes_robotiq_2f140_calibration_adapter" params="prefix">
     <link name="${prefix}base">
       <inertial>
@@ -18,5 +18,5 @@
         <origin xyz="0 0 0" rpy="0 0 0" />
         <geometry>
-          <mesh filename="package://mimik_description/meshes/mimik/ur_mounting_plate/visual/2k.dae"/>
+          <mesh filename="package://oscar_description/meshes/udes/robotiq_2f140_calibration_adapter/visual/928.dae"/>
         </geometry>
         <material name="">
@@ -27,15 +27,8 @@
         <origin xyz="0 0 0" rpy="0 0 0" />
         <geometry>
-          <mesh filename="package://mimik_description/meshes/mimik/ur_mounting_plate/collision/cv12.stl"/>
+          <mesh filename="package://oscar_description/meshes/udes/robotiq_2f140_calibration_adapter/collision/928.stl"/>
         </geometry>
       </collision>
     </link>
-    <link name="${prefix}robotside" />
-    <!-- Mean of multiple points of the surface -->
-    <joint name="${prefix}robotside_joint" type="fixed">
-      <origin xyz="0 0 0.01309" rpy="0 0 0" />
-      <parent link="${prefix}base" />
-      <child link="${prefix}robotside" />
-    </joint>
   </xacro:macro>
 </robot>

File: urdf/udes/ur3_capture_tool_macro.xacro (robot description, xacro)
@@ -1,7 +1,7 @@
 <?xml version="1.0"?>
-<robot name="mimik_pipette_p200" xmlns:xacro="http://www.ros.org/wiki/xacro">
-  <xacro:macro name="mimik_pipette_p200" params="prefix">
+<robot name="udes_ur3_capture_tool" xmlns:xacro="http://www.ros.org/wiki/xacro">
+  <xacro:macro name="udes_ur3_capture_tool" params="prefix">
     <!-- TODO measure or calculate -->
-    <link name="${prefix}base">
+    <link name="${prefix}robotside">
       <inertial>
         <origin xyz="0 0 0" rpy="0 0 0" />
@@ -18,5 +18,5 @@
         <origin xyz="0 0 0" rpy="0 0 0" />
         <geometry>
-          <mesh filename="package://mimik_description/meshes/mimik/pipette_p200/visual/9k.dae"/>
+          <mesh filename="package://oscar_description/meshes/udes/ur3_capture_tool/visual/1k.dae"/>
         </geometry>
         <material name="">
@@ -27,14 +27,13 @@
         <origin xyz="0 0 0" rpy="0 0 0" />
         <geometry>
-          <mesh filename="package://mimik_description/meshes/mimik/pipette_p200/collision/pipette_p200_coarse.stl"/>
+          <mesh filename="package://oscar_description/meshes/udes/ur3_capture_tool/collision/1k.stl"/>
         </geometry>
       </collision>
     </link>
-    <link name="${prefix}tip" />
-    <joint name="${prefix}tip_joint" type="fixed">
-      <!-- Original CAD -->
-      <origin xyz="0.253442 0 0" rpy="0 0 0" />
-      <parent link="${prefix}base" />
-      <child link="${prefix}tip" />
+    <link name="${prefix}tcp" />
+    <joint name="${prefix}tcp_joint" type="fixed">
+      <origin xyz="0.0745 0 0" rpy="0 0 0" />
+      <parent link="${prefix}robotside" />
+      <child link="${prefix}tcp" />
     </joint>
   </xacro:macro>

File: urdf/udes/ur_big_mounting_plate_macro.xacro (robot description, xacro)
@@ -1,5 +1,5 @@
 <?xml version="1.0"?>
-<robot name="mimik_ur_big_mounting_plate" xmlns:xacro="http://www.ros.org/wiki/xacro">
-  <xacro:macro name="mimik_ur_big_mounting_plate" params="prefix">
+<robot name="udes_ur_big_mounting_plate" xmlns:xacro="http://www.ros.org/wiki/xacro">
+  <xacro:macro name="udes_ur_big_mounting_plate" params="prefix">
     <link name="${prefix}base">
       <inertial>
@@ -18,5 +18,5 @@
         <origin xyz="0 0 0" rpy="0 0 0" />
         <geometry>
-          <mesh filename="package://mimik_description/meshes/mimik/ur_big_mounting_plate/visual/171k.dae"/>
+          <mesh filename="package://oscar_description/meshes/udes/ur_big_mounting_plate/visual/171k.dae"/>
         </geometry>
         <material name="">
@@ -27,5 +27,5 @@
         <origin xyz="0 0 0" rpy="0 0 0" />
         <geometry>
-          <mesh filename="package://mimik_description/meshes/mimik/ur_big_mounting_plate/collision/bb12.stl"/>
+          <mesh filename="package://oscar_description/meshes/udes/ur_big_mounting_plate/collision/bb12.stl"/>
         </geometry>
       </collision>

File: urdf/udes/ur_mounting_plate_macro.xacro (robot description, xacro)
@@ -1,9 +1,10 @@
 <?xml version="1.0"?>
-<robot name="newport_vh3660_48x48" xmlns:xacro="http://www.ros.org/wiki/xacro">
-  <xacro:macro name="newport_vh3660_48x48" params="prefix">
+<robot name="udes_ur_mounting_plate" xmlns:xacro="http://www.ros.org/wiki/xacro">
+  <xacro:macro name="udes_ur_mounting_plate" params="prefix">
     <link name="${prefix}base">
       <inertial>
         <origin xyz="0 0 0" rpy="0 0 0" />
-        <mass value="19.86735" />
+        <!-- Not measured -->
+        <mass value="0.5" />
         <inertia
           ixx="0"
@@ -17,5 +18,5 @@
         <origin xyz="0 0 0" rpy="0 0 0" />
         <geometry>
-		<mesh filename="package://oscar_description/meshes/newport/vh3660/visual/82k.dae"/>
+          <mesh filename="package://oscar_description/meshes/udes/ur_mounting_plate/visual/2k.dae"/>
         </geometry>
         <material name="">
@@ -26,14 +27,14 @@
         <origin xyz="0 0 0" rpy="0 0 0" />
         <geometry>
-		<mesh filename="package://oscar_description/meshes/newport/vh3660/collision/bb12.stl"/>
+          <mesh filename="package://oscar_description/meshes/udes/ur_mounting_plate/collision/cv12.stl"/>
         </geometry>
       </collision>
     </link>
-    <link name="${prefix}tabletop" />
-    <joint name="${prefix}tabletop_joint" type="fixed">
-      <!-- Taken from CAD in inches, converted to meters -->
-      <origin xyz="0 0 ${4.3215 * 0.0254}" rpy="0 0 0" />
+    <link name="${prefix}robotside" />
+    <!-- Mean of multiple points of the surface -->
+    <joint name="${prefix}robotside_joint" type="fixed">
+      <origin xyz="0 0 0.01309" rpy="0 0 0" />
       <parent link="${prefix}base" />
-      <child link="${prefix}tabletop" />
+      <child link="${prefix}robotside" />
     </joint>
   </xacro:macro>
