Commit message: [refac] changed tcp to tip

File: urdf/mimik/pipette_p200_macro.xacro (robot description, xacro)
@@ -31,9 +31,10 @@
       </collision>
     </link>
-    <link name="${prefix}tcp" />
-    <joint name="${prefix}tcp_joint" type="fixed">
-      <origin xyz="0.25344 0 0" rpy="0 0 0" />
+    <link name="${prefix}tip" />
+    <joint name="${prefix}tip_joint" type="fixed">
+      <!-- Original CAD -->
+      <origin xyz="0.253442 0 0" rpy="0 0 0" />
       <parent link="${prefix}base" />
-      <child link="${prefix}tcp" />
+      <child link="${prefix}tip" />
     </joint>
   </xacro:macro>

Commit message: [refac] use pipette coarse mesh

File: urdf/mimik/pipette_p200_macro.xacro (robot description, xacro)
@@ -27,5 +27,5 @@
         <origin xyz="0 0 0" rpy="0 0 0" />
         <geometry>
-          <mesh filename="package://mimik_description/meshes/mimik/pipette_p200/collision/p36.stl"/>
+          <mesh filename="package://mimik_description/meshes/mimik/pipette_p200/collision/pipette_p200_coarse.stl"/>
         </geometry>
       </collision>
