Commit message: [refac] drop ur type number

File: urdf/mimik/ur_big_mounting_plate_macro.xacro (robot description, xacro)
@@ -1,5 +1,5 @@
 <?xml version="1.0"?>
-<robot name="mimik_ur3_big_mounting_plate" xmlns:xacro="http://www.ros.org/wiki/xacro">
-  <xacro:macro name="mimik_ur3_big_mounting_plate" params="prefix">
+<robot name="mimik_ur_big_mounting_plate" xmlns:xacro="http://www.ros.org/wiki/xacro">
+  <xacro:macro name="mimik_ur_big_mounting_plate" params="prefix">
     <link name="${prefix}base">
       <inertial>
@@ -18,5 +18,5 @@
         <origin xyz="0 0 0" rpy="0 0 0" />
         <geometry>
-          <mesh filename="package://mimik_description/meshes/mimik/ur3_big_mounting_plate/visual/171k.dae"/>
+          <mesh filename="package://mimik_description/meshes/mimik/ur_big_mounting_plate/visual/171k.dae"/>
         </geometry>
         <material name="">
@@ -27,5 +27,5 @@
         <origin xyz="0 0 0" rpy="0 0 0" />
         <geometry>
-          <mesh filename="package://mimik_description/meshes/mimik/ur3_big_mounting_plate/collision/bb12.stl"/>
+          <mesh filename="package://mimik_description/meshes/mimik/ur_big_mounting_plate/collision/bb12.stl"/>
         </geometry>
       </collision>

File: urdf/mimik/ur_mounting_plate_macro.xacro (robot description, xacro)
@@ -1,5 +1,5 @@
 <?xml version="1.0"?>
-<robot name="mimik_ur3_mounting_plate" xmlns:xacro="http://www.ros.org/wiki/xacro">
-  <xacro:macro name="mimik_ur3_mounting_plate" params="prefix">
+<robot name="mimik_ur_mounting_plate" xmlns:xacro="http://www.ros.org/wiki/xacro">
+  <xacro:macro name="mimik_ur_mounting_plate" params="prefix">
     <link name="${prefix}base">
       <inertial>
@@ -18,5 +18,5 @@
         <origin xyz="0 0 0" rpy="0 0 0" />
         <geometry>
-          <mesh filename="package://mimik_description/meshes/mimik/ur3_mounting_plate/visual/2k.dae"/>
+          <mesh filename="package://mimik_description/meshes/mimik/ur_mounting_plate/visual/2k.dae"/>
         </geometry>
         <material name="">
@@ -27,5 +27,5 @@
         <origin xyz="0 0 0" rpy="0 0 0" />
         <geometry>
-          <mesh filename="package://mimik_description/meshes/mimik/ur3_mounting_plate/collision/cv12.stl"/>
+          <mesh filename="package://mimik_description/meshes/mimik/ur_mounting_plate/collision/cv12.stl"/>
         </geometry>
       </collision>
