Commit message: add markings to tabletop

File: urdf/newport/vh3660_48x48_macro.xacro (robot description, xacro)
@@ -17,5 +17,5 @@
         <origin xyz="0 0 0" rpy="0 0 0" />
         <geometry>
-		<mesh filename="package://mimik_description/meshes/newport/vh3660/visual/70k.dae"/>
+		<mesh filename="package://mimik_description/meshes/newport/vh3660/visual/82k.dae"/>
         </geometry>
         <material name="">
